File: hardware/galdr-carrier.kicad_sch (KiCad schematic)
At the start: 56 parts, among them J1 ESP32-S3 DevBoard, Q1 FQP27P06, U1 BTT TMC2209 V1.3, U2 BTT TMC2209 V1.3, U3 BTT TMC2209 V1.3, U4 BTT TMC2209 V1.3

Commit message: Working on 4th axis
Connections:
- net +3V3: no longer U2.2 (MS1), U3.3 (MS2), U4.2 (MS1), U4.3 (MS2)
- net GND: now also U2.2 (MS1), U3.3 (MS2), U4.2 (MS1), U4.3 (MS2)
- net TMC_BUS: no longer R_UART.2
